File: Board/mainplate.sch (EAGLE design)
At the start: 29 parts, among them U1 M24C04-WMN6P, U2 PCF8563T/F4,118, U3 STM32F103CBT6, X1 22-23-2091, X2 22-23-2041

Commit message: Process commit
Parts:
- added AUDIO_1, AUDIO_2, BTN_IN, BTN_OUT, USB_DM, USB_DP, USB_GND, USB_VCC: (no value), wirepad:2,54/1,0
Connections:
- net N$16 renamed LED_G
- net N$17 renamed LED_R
- removed net N$15: LED_GND.P
- removed net NFC_RESET: U3.PA3
- new net AUDIO_1: AUDIO_1.P
- new net USB_DM: USB_DM.P
- new net USB_DP: USB_DP.P
- new net USB_VCC: USB_VCC.P
- net GND: now also AUDIO_2.P, LED_GND.P, USB_GND.P
- net NFC_RST: now also U3.PA3
- net VBAT: now also BTN_IN.P
- net VBAT2: now also BTN_OUT.P
Changed lines of the file:
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@@
 <part name="LED_G" library="wirepad" deviceset="2,54/1,0" device=""/>
 <part name="LED_GND" library="wirepad" deviceset="2,54/1,0" device=""/>
+<part name="USB_VCC" library="wirepad" deviceset="2,54/1,0" device=""/>
+<part name="USB_DM" library="wirepad" deviceset="2,54/1,0" device=""/>
+<part name="USB_DP" library="wirepad" deviceset="2,54/1,0" device=""/>
+<part name="USB_GND" library="wirepad" deviceset="2,54/1,0" device=""/>
+<part name="BTN_IN" library="wirepad" deviceset="2,54/1,0" device=""/>
+<part name="BTN_OUT" library="wirepad" deviceset="2,54/1,0" device=""/>
+<part name="AUDIO_1" library="wirepad" deviceset="2,54/1,0" device=""/>
+<part name="AUDIO_2" library="wirepad" deviceset="2,54/1,0" device=""/>
 </parts>
 <sheets>
@@
 <instance part="LED_G" gate="P" x="-53.34" y="109.22"/>
 <instance part="LED_GND" gate="P" x="-53.34" y="104.14"/>
+<instance part="USB_VCC" gate="P" x="-53.34" y="93.98"/>
+<instance part="USB_DM" gate="P" x="-53.34" y="88.9"/>
+<instance part="USB_DP" gate="P" x="-53.34" y="83.82"/>
+<instance part="USB_GND" gate="P" x="-53.34" y="78.74"/>
+<instance part="BTN_IN" gate="P" x="-53.34" y="71.12"/>
+<instance part="BTN_OUT" gate="P" x="-53.34" y="66.04"/>
+<instance part="AUDIO_1" gate="P" x="-53.34" y="58.42"/>
+<instance part="AUDIO_2" gate="P" x="-53.34" y="53.34"/>
 </instances>
 <busses>
@@
 <label x="58.42" y="20.32" size="1.778" layer="95" xref="yes"/>
 </segment>
+<segment>
+<pinref part="LED_GND" gate="P" pin="P"/>
+<wire x1="-50.8" y1="104.14" x2="-45.72" y2="104.14" width="0.1524" layer="91"/>
+<label x="-45.72" y="104.14" size="1.778" layer="95" xref="yes"/>
+</segment>
+<segment>
+<pinref part="AUDIO_2" gate="P" pin="P"/>
+<wire x1="-50.8" y1="53.34" x2="-45.72" y2="53.34" width="0.1524" layer="91"/>
+<label x="-45.72" y="53.34" size="1.778" layer="95" xref="yes"/>
+</segment>
+<segment>
+<pinref part="USB_GND" gate="P" pin="P"/>
+<wire x1="-50.8" y1="78.74" x2="-45.72" y2="78.74" width="0.1524" layer="91"/>
+<label x="-45.72" y="78.74" size="1.778" layer="95" xref="yes"/>
+</segment>
 </net>
 <net name="N$3" class="0">
@@
 <junction x="-30.48" y="180.34"/>
 <label x="-33.02" y="180.34" size="1.778" layer="95" rot="R180" xref="yes"/>
+</segment>
+<segment>
+<pinref part="BTN_OUT" gate="P" pin="P"/>
+<wire x1="-50.8" y1="66.04" x2="-45.72" y2="66.04" width="0.1524" layer="91"/>
+<label x="-45.72" y="66.04" size="1.778" layer="95" xref="yes"/>
 </segment>
 </net>
@@
 <label x="205.74" y="48.26" size="1.778" layer="95" rot="R180" xref="yes"/>
 </segment>
-</net>
-<net name="NFC_RESET" class="0">
 <segment>
 <pinref part="U3" gate="A" pin="PA3"/>
@@
 <label x="60.96" y="33.02" size="1.778" layer="95" xref="yes"/>
 </segment>
+<segment>
+<pinref part="BTN_IN" gate="P" pin="P"/>
+<wire x1="-50.8" y1="71.12" x2="-45.72" y2="71.12" width="0.1524" layer="91"/>
+<label x="-45.72" y="71.12" size="1.778" layer="95" xref="yes"/>
+</segment>
 </net>
 <net name="N$13" class="0">
@@
 </segment>
 </net>
-<net name="N$15" class="0">
-<segment>
-<pinref part="LED_GND" gate="P" pin="P"/>
-<wire x1="-50.8" y1="104.14" x2="-38.1" y2="104.14" width="0.1524" layer="91"/>
-</segment>
-</net>
-<net name="N$16" class="0">
+<net name="LED_G" class="0">
 <segment>
 <pinref part="LED_G" gate="P" pin="P"/>
-<wire x1="-50.8" y1="109.22" x2="-40.64" y2="109.22" width="0.1524" layer="91"/>
-<wire x1="-40.64" y1="109.22" x2="-40.64" y2="106.68" width="0.1524" layer="91"/>
-<wire x1="-40.64" y1="106.68" x2="-38.1" y2="106.68" width="0.1524" layer="91"/>
-</segment>
-</net>
-<net name="N$17" class="0">
+<wire x1="-50.8" y1="109.22" x2="-45.72" y2="109.22" width="0.1524" layer="91"/>
+<label x="-45.72" y="109.22" size="1.778" layer="95" xref="yes"/>
+</segment>
+</net>
+<net name="LED_R" class="0">
 <segment>
 <pinref part="LED_R" gate="P" pin="P"/>
-<wire x1="-50.8" y1="114.3" x2="-38.1" y2="114.3" width="0.1524" layer="91"/>
-<wire x1="-38.1" y1="114.3" x2="-38.1" y2="109.22" width="0.1524" layer="91"/>
-</segment>
-</net>
+<wire x1="-50.8" y1="114.3" x2="-45.72" y2="114.3" width="0.1524" layer="91"/>
+<label x="-45.72" y="114.3" size="1.778" layer="95" xref="yes"/>
+</segment>
+</net>
+<net name="AUDIO_1" class="0">
+<segment>
+<pinref part="AUDIO_1" gate="P" pin="P"/>
+<wire x1="-50.8" y1="58.42" x2="-45.72" y2="58.42" width="0.1524" layer="91"/>
+<label x="-45.72" y="58.42" size="1.778" layer="95" xref="yes"/>
+</segment>
+</net>
+<net name="USB_VCC" class="0">
+<segment>
+<pinref part="USB_VCC" gate="P" pin="P"/>
+<wire x1="-50.8" y1="93.98" x2="-45.72" y2="93.98" width="0.1524" layer="91"/>
+<label x="-45.72" y="93.98" size="1.778" layer="95" xref="yes"/>
+</segment>
+</net>
+<net name="USB_DM" class="0">
+<segment>
+<pinref part="USB_DM" gate="P" pin="P"/>
+<wire x1="-50.8" y1="88.9" x2="-45.72" y2="88.9" width="0.1524" layer="91"/>
+<label x="-45.72" y="88.9" size="1.778" layer="95" xref="yes"/>
+</segment>
+</net>
+<net name="USB_DP" class="0">
+<segment>
+<pinref part="USB_DP" gate="P" pin="P"/>
+<wire x1="-50.8" y1="83.82" x2="-45.72" y2="83.82" width="0.1524" layer="91"/>
+<label x="-45.72" y="83.82" size="1.778" layer="95" xref="yes"/>
+</segment>
+</net>

Commit message: plate process
Parts:
- Q2: device crystal-geyer_V1_0:KX-7 -> crystal-geyer_V1_0:KX-K
Changed lines of the file:
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@@
 <?xml version="1.0" encoding="utf-8"?>
 <!DOCTYPE eagle SYSTEM "eagle.dtd">
-<eagle version="8.6.0">
+<eagle version="8.6.3">
 <drawing>
 <settings>
@@
 <part name="U$2" library="Microchip_By_element14_Batch_1" deviceset="MCP73831T-2ACI/OT" device=""/>
 <part name="U2" library="NXP_By_element14_Batch_1" deviceset="PCF8563T/F4,118" device=""/>
-<part name="Q2" library="crystal-geyer_V1_0" deviceset="KX" device="-7"/>
+<part name="Q2" library="crystal-geyer_V1_0" deviceset="KX" device="-K"/>
 <part name="U3" library="ST Microelctronics_By_element14_Batch_1" deviceset="STM32F103CBT6" device=""/>
 <part name="Q1" library="crystal-geyer_V1_0" deviceset="KX-327" device="-NHT"/>

Commit message: First release version
Connections:
- removed net USB: U$2.VDD
- new net N$15: U$2.STAT, U3.PB12
- net AUDIO_1: now also U3.PB3
- net LED_G: now also U3.PC14-OSC32_IN
- net LED_R: now also U3.PC13-TAMPER-RTC
- net USB_DM: now also U3.PA11
- net USB_DP: now also U3.PA12
- net USB_VCC: now also U$2.VDD
Changed lines of the file:
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@@
 <?xml version="1.0" encoding="utf-8"?>
 <!DOCTYPE eagle SYSTEM "eagle.dtd">
-<eagle version="8.6.3">
+<eagle version="8.6.0">
 <drawing>
 <settings>
@@
 <setting verticaltext="up"/>
 </settings>
-<grid distance="0.1" unitdist="inch" unit="inch" style="dots" multiple="1" display="yes" altdistance="0.01" altunitdist="inch" altunit="inch"/>
+<grid distance="0.1" unitdist="inch" unit="inch" style="lines" multiple="1" display="no" altdistance="0.01" altunitdist="inch" altunit="inch"/>
 <layers>
 <layer number="1" name="Top" color="4" fill="10" visible="no" active="no"/>
@@
 <pinref part="U3" gate="A" pin="BOOT0"/>
 <wire x1="160.02" y1="121.92" x2="162.56" y2="121.92" width="0.1524" layer="91"/>
-<wire x1="162.56" y1="121.92" x2="162.56" y2="101.6" width="0.1524" layer="91"/>
-<wire x1="162.56" y1="101.6" x2="165.1" y2="101.6" width="0.1524" layer="91"/>
-<label x="165.1" y="101.6" size="1.778" layer="95" xref="yes"/>
+<wire x1="162.56" y1="121.92" x2="162.56" y2="99.06" width="0.1524" layer="91"/>
+<wire x1="162.56" y1="99.06" x2="165.1" y2="99.06" width="0.1524" layer="91"/>
+<label x="165.1" y="99.06" size="1.778" layer="95" xref="yes"/>
 </segment>
 <segment>
@@
 </segment>
 </net>
-<net name="USB" class="0">
-<segment>
-<pinref part="U$2" gate="A" pin="VDD"/>
-<wire x1="17.78" y1="38.1" x2="2.54" y2="38.1" width="0.1524" layer="91"/>
-<label x="2.54" y="38.1" size="1.778" layer="95" rot="R180" xref="yes"/>
-</segment>
-</net>
 <net name="N$1" class="0">
 <segment>
 <pinref part="Q2" gate="G$1" pin="2"/>
-<wire x1="173.228" y1="118.11" x2="173.228" y2="121.92" width="0.1524" layer="91"/>
-<wire x1="173.228" y1="121.92" x2="167.64" y2="121.92" width="0.1524" layer="91"/>
-<wire x1="167.64" y1="121.92" x2="167.64" y2="116.84" width="0.1524" layer="91"/>
+<wire x1="173.228" y1="118.11" x2="173.228" y2="119.38" width="0.1524" layer="91"/>
+<wire x1="173.228" y1="119.38" x2="167.64" y2="119.38" width="0.1524" layer="91"/>
+<wire x1="167.64" y1="119.38" x2="167.64" y2="116.84" width="0.1524" layer="91"/>
 <pinref part="U3" gate="A" pin="PD0-OSC_IN"/>
 <wire x1="167.64" y1="116.84" x2="160.02" y2="116.84" width="0.1524" layer="91"/>
@@
 <segment>
 <pinref part="Q2" gate="G$1" pin="1"/>
-<wire x1="173.228" y1="113.03" x2="173.228" y2="109.22" width="0.1524" layer="91"/>
-<wire x1="173.228" y1="109.22" x2="167.64" y2="109.22" width="0.1524" layer="91"/>
-<wire x1="167.64" y1="109.22" x2="167.64" y2="114.3" width="0.1524" layer="91"/>
+<wire x1="173.228" y1="113.03" x2="173.228" y2="111.76" width="0.1524" layer="91"/>
+<wire x1="173.228" y1="111.76" x2="167.64" y2="111.76" width="0.1524" layer="91"/>
+<wire x1="167.64" y1="111.76" x2="167.64" y2="114.3" width="0.1524" layer="91"/>
 <pinref part="U3" gate="A" pin="PD1-OSC_OUT"/>
 <wire x1="167.64" y1="114.3" x2="160.02" y2="114.3" width="0.1524" layer="91"/>
@@
 <label x="-45.72" y="109.22" size="1.778" layer="95" xref="yes"/>
 </segment>
+<segment>
+<pinref part="U3" gate="A" pin="PC14-OSC32_IN"/>
+<wire x1="160.02" y1="106.68" x2="165.1" y2="106.68" width="0.1524" layer="91"/>
+<label x="165.1" y="106.68" size="1.778" layer="95" xref="yes"/>
+</segment>
 </net>
 <net name="LED_R" class="0">
@@
 <label x="-45.72" y="114.3" size="1.778" layer="95" xref="yes"/>
 </segment>
+<segment>
+<pinref part="U3" gate="A" pin="PC13-TAMPER-RTC"/>
+<wire x1="160.02" y1="109.22" x2="177.8" y2="109.22" width="0.1524" layer="91"/>
+<label x="177.8" y="109.22" size="1.778" layer="95" xref="yes"/>
+</segment>
 </net>
 <net name="AUDIO_1" class="0">
@@
 <label x="-45.72" y="58.42" size="1.778" layer="95" xref="yes"/>
 </segment>
+<segment>
+<pinref part="U3" gate="A" pin="PB3"/>
+<wire x1="104.14" y1="101.6" x2="101.6" y2="101.6" width="0.1524" layer="91"/>
+<label x="101.6" y="101.6" size="1.778" layer="95" rot="R180" xref="yes"/>
+</segment>
 </net>
 <net name="USB_VCC" class="0">
@@
 <label x="-45.72" y="93.98" size="1.778" layer="95" xref="yes"/>
 </segment>
+<segment>
+<pinref part="U$2" gate="A" pin="VDD"/>
+<wire x1="17.78" y1="38.1" x2="2.54" y2="38.1" width="0.1524" layer="91"/>
+<label x="2.54" y="38.1" size="1.778" layer="95" rot="R180" xref="yes"/>
+</segment>
 </net>
 <net name="USB_DM" class="0">
@@
 <label x="-45.72" y="88.9" size="1.778" layer="95" xref="yes"/>
 </segment>
+<segment>
+<pinref part="U3" gate="A" pin="PA11"/>
+<wire x1="104.14" y1="38.1" x2="81.28" y2="38.1" width="0.1524" layer="91"/>
+<label x="81.28" y="38.1" size="1.778" layer="95" rot="R180" xref="yes"/>
+</segment>
 </net>
 <net name="USB_DP" class="0">
@@
 <label x="-45.72" y="83.82" size="1.778" layer="95" xref="yes"/>
 </segment>
-</net>
+<segment>
+<pinref part="U3" gate="A" pin="PA12"/>
+<wire x1="104.14" y1="35.56" x2="99.06" y2="35.56" width="0.1524" layer="91"/>
+<label x="99.06" y="35.56" size="1.778" layer="95" rot="R180" xref="yes"/>
+</segment>
+</net>
+<net name="N$15" class="0">
+<segment>
+<pinref part="U$2" gate="A" pin="STAT"/>
+<wire x1="53.34" y1="38.1" x2="58.42" y2="38.1" width="0.1524" layer="91"/>
+<wire x1="58.42" y1="38.1" x2="58.42" y2="71.12" width="0.1524" layer="91"/>
+<wire x1="58.42" y1="71.12" x2="88.9" y2="71.12" width="0.1524" layer="91"/>
+<wire x1="88.9" y1="71.12" x2="88.9" y2="78.74" width="0.1524" layer="91"/>
+<pinref part="U3" gate="A" pin="PB12"/>
+<wire x1="88.9" y1="78.74" x2="104.14" y2="78.74" width="0.1524" layer="91"/>
+</segment>
+</net>
